Commit message: 'perfect' odometry and removed workarounds

File: src/simulation/description/robot.urdf.xacro (robot description, xacro)
@@ -2,8 +2,11 @@
 <robot xmlns:xacro="http://www.ros.org/wiki/xacro"  name="robot">
     <!-- ROVER PARAMETERS-->
+    <xacro:property name="package_name" value="simulation" />
     <!-- wheel parameters -->
     <xacro:property name="wheel_radius" value="0.05" />
     <xacro:property name="wheel_width" value="0.05" />
     <xacro:property name="wheel_mass" value="0.1" />
+    <xacro:property name="wheel_mu1" value="10.0" />
+    <xacro:property name="wheel_mu2" value="10.0" />
     <!-- caster parameters -->
     <xacro:property name="caster_radius" value="0.05" />
@@ -22,4 +25,3 @@
     <xacro:include filename="robot_core.xacro" />
     <xacro:include filename="ros2_control.xacro" />
-    <xacro:include filename="gazebo_plugins.xacro" />
 </robot>

File: src/simulation/description/robot_core.xacro (robot description, xacro)
@@ -16,4 +16,9 @@
     <!-- BASE LINK -->
     <link name="base_link">
+        <inertial>
+            <mass value="0.0001"/>
+            <inertia ixx="0.000001" ixy="0.0" ixz="0.0" iyy="0.000001" iyz="0.0" izz="0.000001"/>
+            <origin xyz="0 0 0" rpy="0 0 0"/>
+          </inertial>
     </link>
     <!-- CHASSIS LINK -->
@@ -69,4 +74,6 @@
     <gazebo reference="left_wheel">
         <material>Gazebo/Blue</material>
+        <mu1 value="${wheel_mu1}"/>
+        <mu2 value="${wheel_mu2}"/>
     </gazebo>
     <!-- RIGHT WHEEL LINK -->
@@ -95,4 +102,6 @@
     <gazebo reference="right_wheel">
         <material>Gazebo/Blue</material>
+        <mu1 value="${wheel_mu1}"/>
+        <mu2 value="${wheel_mu2}"/>
     </gazebo>
     <!-- CASTER WHEEL LINK -->

File: src/simulation/description/ros2_control.xacro (robot description, xacro)
@@ -24,20 +24,8 @@
 <gazebo>
     <plugin name="ign_ros2_control::IgnitionROS2ControlPlugin" filename="ign_ros2_control-system">
-        <parameters>$(find my_bot)/config/controllers.yaml </parameters>
+        <parameters>$(find ${package_name})/config/controllers.yaml </parameters>
         <controller_manager_prefix_node_name>controller_manager</controller_manager_prefix_node_name>
         <robotNamespace>/robot</robotNamespace>
     </plugin>
-    <!-- Publish ground truth pose -->
-    <plugin name="ignition::gazebo::systems::PosePublisher" filename="libignition-gazebo-pose-publisher-system.so">
-        <!-- <publish_link_pose>true</publish_link_pose> -->
-        <!-- <publish_sensor_pose>true</publish_sensor_pose> -->
-        <!-- <publish_collision_pose>false</publish_collision_pose> -->
-        <!-- <publish_visual_pose>false</publish_visual_pose> -->
-        <!-- <publish_model_pose>true</publish_model_pose> -->
-        <publish_nested_model_pose>true</publish_nested_model_pose>
-        <use_pose_vector_msg>true</use_pose_vector_msg>
-        <!-- <static_publisher>true</static_publisher> -->
-        <static_update_frequency>-1</static_update_frequency>
-    </plugin>
 </gazebo>
 </robot>
