Commit message: Added lidar to the rolly boi

File: src/simulation/description/gazebo_plugins.xacro (robot description, xacro)
@@ -8,4 +8,11 @@
             <render_engine>ogre2</render_engine>
         </plugin>
+        <!-- <plugin name="laser_controller" filename="libgazebo_ros_ray_sensor.so">
+            <ros>
+                <argument>~/out:=scan</argument>
+            </ros>
+            <output_type>sensor_msgs/LaserScan</output_type>
+            <frame_name>laser_frame</frame_name>
+        </plugin> -->
     </gazebo>
 </robot>

File: src/simulation/description/lidar.xacro (robot description, xacro)
@@ -4,21 +4,7 @@
         <parent link="chassis"/>
         <child link="laser_frame"/>
-        <origin xyz="${chassis_length/2} 0 ${chassis_height/2}" rpy="0 0 0"/>
+        <origin xyz="${chassis_length+lidar_viz_cylinder_radius*2} 0 ${chassis_height}" rpy="0 0 0"/>
     </joint>
     <link name="laser_frame">
-        <visual>
-            <geometry>
-                <cylinder radius="0.05" length="0.04"/>
-            </geometry>
-            <material name="red"/>
-        </visual>
-        <collision>
-            <geometry>
-                <cylinder radius="0.05" length="0.04"/>
-            </geometry>
-        </collision>
-        <xacro:inertial_cylinder mass="0.1" length="0.04" radius="0.05">
-            <origin xyz="0 0 0" rpy="0 0 0"/>
-        </xacro:inertial_cylinder>
     </link>
     <gazebo reference="laser_frame">
@@ -38,6 +24,6 @@
                         <samples>1</samples>
                         <resolution>0.01</resolution>
-                        <min_angle>${-lidar_vfov/2}</min_angle>
-                        <max_angle>${lidar_vfov/2}</max_angle>
+                        <min_angle>-0.01</min_angle>
+                        <max_angle>0.01</max_angle>
                     </vertical>
                 </scan>

File: src/simulation/description/robot.urdf.xacro (robot description, xacro)
@@ -26,4 +26,6 @@
     <xacro:property name="lidar_max_range" value="30" />
     <xacro:property name="lidar_update_rate" value="1" />
+    <xacro:property name="lidar_viz_cylinder_radius" value="0.01" />
+    <xacro:property name="lidar_viz_cylinder_height" value="0.01" />
     <!-- dynamic parameters -->
     <xacro:property name="wheel_max_velocity" value="10" />
