Commit message: causing merge conflicts because that is fun

File: src/my_bot/description/gazebo_plugins.xacro (robot description, xacro)
@@ -8,5 +8,5 @@
             <!-- <publish_collision_pose>false</publish_collision_pose> -->
             <!-- <publish_visual_pose>false</publish_visual_pose> -->
-            <!-- <publish_model_pose>true</publish_model_pose> -->
+            <publish_model_pose>true</publish_model_pose>
             <publish_nested_model_pose>true</publish_nested_model_pose>
             <use_pose_vector_msg>true</use_pose_vector_msg>
@@ -14,4 +14,10 @@
             <static_update_frequency>-1</static_update_frequency>
         </plugin>
+        <!-- Plugin for the lidar sensor -->
+        <plugin
+            filename="libignition-gazebo-sensors-system.so"
+            name="ignition::gazebo::systems::Sensors">
+            <render_engine>ogre2</render_engine>
+        </plugin>
     </gazebo>
 </robot>

File: src/my_bot/description/robot.urdf.xacro (robot description, xacro)
@@ -18,4 +18,9 @@
     <xacro:property name="chassis_position" value="-0.1" />
     <xacro:property name="chassis_mass" value="0.5" />
+    <!-- lidar parameters -->
+    <xacro:property name="lidar_hfov" value="3.14" />
+    <xacro:property name="lidar_vfov" value="0.3" />
+    <xacro:property name="lidar_max_range" value="30" />
+    <xacro:property name="lidar_update_rate" value="1" />
     <!-- dynamic parameters -->
     <xacro:property name="wheel_max_velocity" value="10" />
@@ -23,3 +28,4 @@
     <xacro:include filename="ros2_control.xacro" />
     <xacro:include filename="gazebo_plugins.xacro" />
+    <xacro:include filename="lidar.xacro" />
 </robot>

File: src/my_bot/description/robot_core.xacro (robot description, xacro)
@@ -13,4 +13,7 @@
     <material name="black">
         <color rgba="0 0 0 1"/>
+    </material>
+    <material name="red">
+        <color rgba="1 0 0 1"/>
     </material>
     <!-- BASE LINK -->
